File: analog_sw2.kicad_pcb (KiCad board)
At the start: 2 copper layers, 70 parts, among them J1 Conn_01x05, J10 Conn_01x05, J11 Conn_01x05, J12 Conn_01x05, J13 Conn_01x05, J14 Conn_01x05, J15 Conn_01x05, J16 Conn_01x05, J17 Conn_01x16, J18 Conn_01x16, J2 Conn_01x05, J3 Conn_01x05, J4 Conn_01x05, J5 Conn_01x05, J6 Conn_01x05, J7 Conn_01x05, J8 Conn_01x05, J9 Conn_01x05, U1 TC4S6FF, U10 TC4S6FF, U11 TC4S6FF, U12 TC4S6FF, U13 TC4S6FF, U14 TC4S6FF, U15 TC4S6FF, U16 TC4S6FF, U17 74HC595, U18 74HC595, U2 TC4S6FF, U3 TC4S6FF, U4 TC4S6FF, U5 TC4S6FF, U6 TC4S6FF, U7 TC4S6FF, U8 TC4S6FF, U9 TC4S6FF

Commit message: update
Parts:
- added P1: , , F.Cu at (171.4, 63.5)
- added P2: , , F.Cu at (171.4, 74.9)
- added P3: , , F.Cu at (171.4, 92.7)
- added P4: , , F.Cu at (171.4, 110.5)
- added P5: , , F.Cu at (171.4, 121.9)
- added P6: , , F.Cu at (185.4, 74.9)
- added P7: , , F.Cu at (185.4, 92.7)
- added P8: NEJI_2.6mm, MyLibrary:NEJI_2.6mm, F.Cu at (185.4, 110.5)
- added REF**: NEJI_2.6mm, MyLibrary:NEJI_2.6mm, F.Cu at (138.4, 62.2)
- added REF**: NEJI_2.6mm, MyLibrary:NEJI_2.6mm, F.Cu at (166.4, 123.2)
- added REF**: NEJI_2.6mm, MyLibrary:NEJI_2.6mm, F.Cu at (166.4, 62.2)
- added REF**: NEJI_2.6mm, MyLibrary:NEJI_2.6mm, F.Cu at (138.4, 123.2)
- C1, C2, R1, R10, R11, R12, R13, R14, R15, R16, R2, R3, R4, R5, R6, R7, R8, R9: moved to B.Cu
- moved D5 149.8 mm to (191.8, 80.0)
- moved D11 146.7 mm to (191.8, 102.9)
- moved D15 135.2 mm to (191.8, 120.7)
- moved R2 130.6 mm to (191.8, 64.8)
- moved D16 128.7 mm to (191.8, 123.2)
- moved R1 126.7 mm to (191.8, 62.2)
- moved R15 126.1 mm to (191.8, 120.7)
- moved D6 124.8 mm to (191.8, 82.5)
- moved D7 120.5 mm to (191.8, 85.1)
- moved R14 118.7 mm to (191.8, 118.1)
- moved D12 118.3 mm to (191.8, 105.4)
- moved D1 118.0 mm to (191.8, 62.2)
- moved R4 117.6 mm to (191.8, 69.8)
- moved D2 117.5 mm to (191.8, 64.8)
- moved R16 115.7 mm to (191.8, 123.2)
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Routing:
- net VCC: track 0.00 -> 174.3 mm, vias 0 -> 1
- net GND3: track 0.00 -> 72.1 mm
- net GND1: track 0.00 -> 72.0 mm
- net GNDA: track 0.00 -> 71.9 mm
- net GND2: track 0.00 -> 68.3 mm
- net GND: track 0.00 -> 52.8 mm, vias 0 -> 10
- net _RCLK: track 0.00 -> 47.7 mm
- net _SRCLK: track 0.00 -> 45.6 mm
- net _SER: track 0.00 -> 20.8 mm
- net _K1: track 0.00 -> 18.9 mm
- net +3.3VDAC: track 0.00 -> 18.3 mm, vias 0 -> 4
- net +3.3VADC: track 0.00 -> 18.3 mm, vias 0 -> 4
- net +3.3VA: track 0.00 -> 18.3 mm, vias 0 -> 4
- net +3.3V: track 0.00 -> 18.2 mm, vias 0 -> 4
- net _K9: track 0.00 -> 17.5 mm
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- added copper zone on B.Cu, net +3.3V
- added copper zone on B.Cu, net +3.3VA
- added copper zone on B.Cu, net +3.3VADC
- added copper zone on B.Cu, net +3.3VDAC
- added copper zone on B.Cu, net GND
- added copper zone on F.Cu, net GND
- added copper zone on F.Cu, net GND1
- added copper zone on F.Cu, net GND2
- added copper zone on F.Cu, net GND3
- added copper zone on F.Cu, net GNDA
Other:
- board outline added: 62.2 x 68.6 mm
- board text added: "GND"
- board text added: "RCLK"
- board text added: "SER"
- board text added: "SRCLK"
- board text added: "VCC"

Commit message: update
Parts:
- added J19: Conn_01x01, Connector_PinHeader_2.54mm:PinHeader_1x01_P2.54mm_Vertical, F.Cu at (167.6, 114.3)
- added J20: Conn_01x01, Connector_PinHeader_2.54mm:PinHeader_1x01_P2.54mm_Vertical, F.Cu at (167.6, 71.1)
- added J21: Conn_01x01, Connector_PinHeader_2.54mm:PinHeader_1x01_P2.54mm_Vertical, F.Cu at (137.2, 71.1)
- added J22: Conn_01x01, Connector_PinHeader_2.54mm:PinHeader_1x01_P2.54mm_Vertical, F.Cu at (137.2, 114.3)
- U17, U18: footprint 74HC:DIP_74HC595 -> Package_SO:SOP-16_4.55x10.3mm_P1.27mm
- moved C2 28.0 mm to (152.4, 111.8), turned to 180 degrees
- moved C1 25.4 mm to (152.4, 81.3), turned to 180 degrees
- moved J12 3.82 mm to (142.2, 110.5)
- moved J16 3.82 mm to (162.6, 110.5)
- moved U17 3.81 mm to (152.4, 77.5)
- moved U18 3.81 mm to (152.4, 108.0)
- moved J13 3.80 mm to (162.6, 64.8)
- moved J9 3.80 mm to (142.2, 64.8)
- moved J11 1.28 mm to (142.2, 95.2)
- moved J15 1.28 mm to (162.6, 95.3)
- moved J10 1.26 mm to (142.2, 80.0)
- moved J14 1.26 mm to (162.6, 80.0)
- moved J5 0.17 mm to (195.6, 61.0)
Connections:
- J17 pad 10: unconnected-(J17-Pad10) -> GND
- J17 pad 11: unconnected-(J17-Pad11) -> GND
- J17 pad 12: unconnected-(J17-Pad12) -> GND
- J17 pad 13: unconnected-(J17-Pad13) -> GND
- J17 pad 14: unconnected-(J17-Pad14) -> GND
- J17 pad 15: unconnected-(J17-Pad15) -> GND
- J17 pad 16: unconnected-(J17-Pad16) -> GND
- J17 pad 8: unconnected-(J17-Pad8) -> GND
- J17 pad 9: unconnected-(J17-Pad9) -> GND
- U17 pad 10: GND -> VCC
- U17 pad 13: VCC -> GND
- U18 pad 10: GND -> VCC
- U18 pad 13: VCC -> GND
Routing:
- net VCC: track 174.3 -> 108.4 mm, vias 1 -> 2
- net GND: track 52.8 -> 18.8 mm, vias 10 -> 15
- net _SRCLK: track 45.6 -> 64.7 mm
- net Net-(U17-QH'): track 11.8 -> 27.1 mm
- net _RCLK: track 47.7 -> 56.0 mm, vias 0 -> 1
- net _K8: track 6.72 -> 14.6 mm
- net _K7: track 6.72 -> 13.3 mm
- net _K13: track 16.5 -> 10.8 mm
- net _K6: track 6.72 -> 12.0 mm
- net _K14: track 16.5 -> 12.0 mm
- net _K5: track 6.72 -> 10.8 mm
- net _S13: track 12.3 -> 8.83 mm
- net _K15: track 16.5 -> 13.3 mm
- net _S14: track 12.3 -> 9.20 mm
- net _S1: track 14.8 -> 11.7 mm
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Other:
- board text added: "(X)"
