File: analog_sw2.kicad_sch (KiCad schematic)
At the start: 70 parts, among them J1 Conn_01x05, J10 Conn_01x05, J11 Conn_01x05, J12 Conn_01x05, J13 Conn_01x05, J14 Conn_01x05, J15 Conn_01x05, J16 Conn_01x05, J17 Conn_01x16, J18 Conn_01x16, J2 Conn_01x05, J3 Conn_01x05, J4 Conn_01x05, J5 Conn_01x05, J6 Conn_01x05, J7 Conn_01x05, J8 Conn_01x05, J9 Conn_01x05, U1 TC4S6FF, U10 TC4S6FF, U11 TC4S6FF, U12 TC4S6FF, U13 TC4S6FF, U14 TC4S6FF, U15 TC4S6FF, U16 TC4S6FF, U17 74HC595, U18 74HC595, U2 TC4S6FF, U3 TC4S6FF, U4 TC4S6FF, U5 TC4S6FF, U6 TC4S6FF, U7 TC4S6FF, U8 TC4S6FF, U9 TC4S6FF

Commit message: update
Parts:
- added J19, J20, J21, J22: Conn_01x01, Connector_PinHeader_2.54mm:PinHeader_1x01_P2.54mm_Vertical, symbol Connector_Generic:Conn_01x01
- U17, U18: footprint 74HC:DIP_74HC595 -> Package_SO:SOP-16_4.55x10.3mm_P1.27mm
Connections:
- net GND: now also J17.10 (Pin_10), J17.11 (Pin_11), J17.12 (Pin_12), J17.13 (Pin_13), J17.14 (Pin_14), J17.15 (Pin_15), J17.16 (Pin_16), J17.8 (Pin_8), J17.9 (Pin_9), U17.13 (~{OE}), U18.13 (~{OE}), J19.1 (Pin_1), J20.1 (Pin_1), J21.1 (Pin_1), J22.1 (Pin_1); no longer U17.10 (~{SRCLR}), U18.10 (~{SRCLR})
- net VCC: now also U17.10 (~{SRCLR}), U18.10 (~{SRCLR}); no longer U17.13 (~{OE}), U18.13 (~{OE})
- no-connect marks 12 -> 3
